File: hardware/boards/pcb-a/pcb-a.kicad_pcb (KiCad board)
At the start: 2 copper layers, 0 parts

Commit message: hw(boards): PCB-F and PCB-K2 placed and routed, DRC 0/0/0 with schematic parity
Placement from panel-coordinates.csv (shared frame for all boards), Brain
board tools reused (route_board/finish_routing/add_gnd_escapes/pours/fields),
plus sync_from_netlist.py (MCP sync drops the '/' net prefix and BOM attrs)
and build.sh to rebuild a board end to end. LED-window DRC rule copied
from the Brain's PCB-K.

Co-Authored-By: Claude Opus 5.5 <noreply@anthropic.com>
Parts:
- added C1: 100nF, Capacitor_SMD:C_0603_1608Metric, F.Cu at (0.00, 0.00)
- added C10, C11, C12, C13, C14, C15, C16, C17, C18, C19, C20, C21, C22, C23, C24, C25: 10nF, Capacitor_SMD:C_0603_1608Metric, F.Cu at (0.00, 0.00)
- added C2: 10uF, Capacitor_SMD:C_0805_2012Metric, F.Cu at (0.00, 0.00)
- added H1, H2, H3, H4: M3, MountingHole:MountingHole_3.2mm_M3, F.Cu at (0.00, 0.00)
- added J1: to carrier J5 (IDC 2x15), Connector_IDC:IDC-Header_2x15_P2.54mm_Vertical, F.Cu at (0.00, 0.00)
- added J2: I2C in (JST-SH 4, Qwiic), Connector_JST:JST_SH_SM04B-SRSS-TB_1x04-1MP_P1.00mm_Horizontal, F.Cu at (0.00, 0.00)
- added J3: to PCB-F (JST-SH 6), Connector_JST:JST_SH_SM06B-SRSS-TB_1x06-1MP_P1.00mm_Horizontal, F.Cu at (0.00, 0.00)
- added J4: to PCB-K1 (JST-SH 10), Connector_JST:JST_SH_SM10B-SRSS-TB_1x10-1MP_P1.00mm_Horizontal, F.Cu at (0.00, 0.00)
- added R1, R2: 4.7k, Resistor_SMD:R_0603_1608Metric, F.Cu at (0.00, 0.00)
- added RE1, RE2, RE3, RE4, RE5, RE6, RE7, RE8: EC11, Rotary_Encoder:RotaryEncoder_Alps_EC11E-Switch_Vertical_H20mm, F.Cu at (0.00, 0.00)
- added U1: MCP23017-E/SO, Package_SO:SOIC-28W_7.5x17.9mm_P1.27mm, F.Cu at (0.00, 0.00)

Commit message: hw(boards): all panel boards routed to DRC 0/0/0, add PCB-S shield adapter, fab outputs
PCB-A, PCB-F, PCB-K1, PCB-K2 and the new PCB-S pass DRC with schematic parity and ERC.
Single-sided bottom assembly; PCB-S ships bare (hand-soldered).

- PCB-A: MCP23017 0x20 moved to SSOP-28 in the front band between E4 and E5; J4 (to PCB-K1)
  moved to the tab next to J1 (cable ~20-25 cm) so the bus stays off the encoder strip;
  strip front edge 99 -> 97.5; H4 onto the tab.
- PCB-K1: MCP 0x21 pins reordered for a planar fan-out; U1 is SSOP-28; J2 over U2.
- PCB-S: shield adapter for the carrier's J15/J16 (I2C -> JST-SH 4, Serial5 -> JST-PH 4 to the M4).
- tools: grid router now sees footprint Edge.Cuts windows and exact pad keep-outs; finish_routing
  routes shortest-first, joins split nets and rips up endpoint blockers; new repair_routes.py and
  tie_loose_gnd.py; GND escapes respect the real outline; sync_from_netlist re-assigns pad nets;
  export_fab groups BOM lines per part and covers PCB-S.
- fab/: Gerbers, BOM and CPL per board for JLCPCB.

Co-Authored-By: Claude Sonnet 5.5 <noreply@anthropic.com>
Parts:
- C1, C10, C11, C12, C13, C14, C15, C16, C17, C18, C19, C2, C20, C21, C22, C23, C24, C25, J1, J2, J3, J4, R1, R2: moved to B.Cu
- U1: value MCP23017-E/SO -> MCP23017T-E/SS; footprint Package_SO:SOIC-28W_7.5x17.9mm_P1.27mm -> Package_SO:SSOP-28_5.3x10.2mm_P0.65mm; moved to B.Cu
- moved J1 317.4 mm to (215.7, 232.8)
- moved J3 313.5 mm to (205.5, 236.7), turned to 180 degrees
- moved J2 306.0 mm to (194.0, 236.7), turned to 180 degrees
- moved R2 298.2 mm to (203.5, 218.0), turned to 90 degrees
- moved H4 297.8 mm to (194.0, 226.0)
- moved R1 296.5 mm to (201.0, 218.0), turned to 90 degrees
- moved C2 286.7 mm to (203.5, 202.0), turned to 90 degrees
- moved J4 283.4 mm to (190.3, 210.0), turned to 90 degrees
- moved C25 279.5 mm to (212.5, 181.5)
- moved C24 276.2 mm to (212.5, 176.5)
- moved RE8 273.9 mm to (209.5, 176.5)
- moved C23 260.2 mm to (186.5, 181.5)
- moved C22 256.8 mm to (186.5, 176.5)
- moved RE7 254.6 mm to (183.5, 176.5)
- moved C21 242.3 mm to (160.5, 181.5)
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Connections:
- net +3V3 renamed /+3V3
- net +5V renamed /+5V
- net ENC1_A renamed /ENC1_A
- net ENC1_B renamed /ENC1_B
- net ENC2_A renamed /ENC2_A
- net ENC2_B renamed /ENC2_B
- net ENC3_A renamed /ENC3_A
- net ENC3_B renamed /ENC3_B
- net ENC4_A renamed /ENC4_A
- net ENC4_B renamed /ENC4_B
- net ENC5_A renamed /ENC5_A
- net ENC5_B renamed /ENC5_B
- net ENC6_A renamed /ENC6_A
- net ENC6_B renamed /ENC6_B
- net ENC7_A renamed /ENC7_A
- net ENC7_B renamed /ENC7_B
- net ENC8_A renamed /ENC8_A
- net ENC8_B renamed /ENC8_B
- net FADER1 renamed /FADER1
- net FADER2 renamed /FADER2
- net FADER3 renamed /FADER3
- net FADER4 renamed /FADER4
- net GND renamed /GND
- net INT_A renamed /INT_A
- net INT_K renamed /INT_K
- net LED_DIN renamed /LED_DIN
- net SCL renamed /SCL
- net SDA renamed /SDA
- J1 pad 18: (no net) -> unconnected-(J1-Pin_18-Pad18)
- RE1 pad S1: ENC1_SW -> /ENC1_SW
- RE2 pad S1: ENC2_SW -> /ENC2_SW
- RE3 pad S1: ENC3_SW -> /ENC3_SW
- RE4 pad S1: ENC4_SW -> /ENC4_SW
- RE5 pad S1: ENC5_SW -> /ENC5_SW
- RE6 pad S1: ENC6_SW -> /ENC6_SW
- RE7 pad S1: ENC7_SW -> /ENC7_SW
- RE8 pad S1: ENC8_SW -> /ENC8_SW
- U1 pad 1: ENC8_SW -> /ENC1_SW
- U1 pad 11: (no net) -> unconnected-(U1-NC-Pad11)
- U1 pad 14: (no net) -> unconnected-(U1-NC-Pad14)
- U1 pad 19: (no net) -> unconnected-(U1-INTB-Pad19)
- U1 pad 2: (no net) -> /ENC2_SW
- U1 pad 21: ENC1_SW -> /ENC5_SW
- U1 pad 22: ENC2_SW -> /ENC6_SW
- U1 pad 23: ENC3_SW -> /ENC7_SW
- U1 pad 24: ENC4_SW -> /ENC8_SW
- U1 pad 25: ENC5_SW -> unconnected-(U1-GPA4-Pad25)
- U1 pad 26: ENC6_SW -> unconnected-(U1-GPA5-Pad26)
- U1 pad 27: ENC7_SW -> unconnected-(U1-GPA6-Pad27)
- U1 pad 28: (no net) -> unconnected-(U1-GPA7-Pad28)
- U1 pad 3: (no net) -> /ENC3_SW
- U1 pad 4: (no net) -> /ENC4_SW
- U1 pad 5: (no net) -> unconnected-(U1-GPB4-Pad5)
- U1 pad 6: (no net) -> unconnected-(U1-GPB5-Pad6)
- U1 pad 7: (no net) -> unconnected-(U1-GPB6-Pad7)
- U1 pad 8: (no net) -> unconnected-(U1-GPB7-Pad8)
Routing:
- net /+3V3: track 0.00 -> 349.5 mm, vias 0 -> 6
- net /ENC1_B: track 0.00 -> 324.1 mm, vias 0 -> 18
- net /ENC3_B: track 0.00 -> 261.6 mm, vias 0 -> 14
- net /ENC3_A: track 0.00 -> 260.6 mm, vias 0 -> 8
- net /ENC2_A: track 0.00 -> 253.7 mm, vias 0 -> 5
- net /ENC1_A: track 0.00 -> 241.4 mm, vias 0 -> 3
- net /ENC2_B: track 0.00 -> 223.1 mm, vias 0 -> 2
- net /ENC4_A: track 0.00 -> 159.7 mm
- net /ENC4_B: track 0.00 -> 157.2 mm
- net /ENC5_A: track 0.00 -> 130.1 mm, vias 0 -> 1
- net /SCL: track 0.00 -> 127.9 mm, vias 0 -> 4
- net /SDA: track 0.00 -> 126.4 mm, vias 0 -> 8
- net /ENC8_SW: track 0.00 -> 103.0 mm, vias 0 -> 1
- net /INT_A: track 0.00 -> 99.9 mm, vias 0 -> 3
- net /ENC5_B: track 0.00 -> 96.8 mm, vias 0 -> 3
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- added copper zone on B.Cu, net /GND
- added copper zone on F.Cu, net /GND
Other:
- board outline added: 217 x 69.6 mm
