File: hardware/boards/pcb-f/pcb-f.kicad_pcb (KiCad board)
At the start: 2 copper layers, 0 parts

Commit message: hw(boards): PCB-F and PCB-K2 placed and routed, DRC 0/0/0 with schematic parity
Placement from panel-coordinates.csv (shared frame for all boards), Brain
board tools reused (route_board/finish_routing/add_gnd_escapes/pours/fields),
plus sync_from_netlist.py (MCP sync drops the '/' net prefix and BOM attrs)
and build.sh to rebuild a board end to end. LED-window DRC rule copied
from the Brain's PCB-K.

Co-Authored-By: Claude Opus 5.5 <noreply@anthropic.com>
Parts:
- added C1: 100nF, Capacitor_SMD:C_0603_1608Metric, B.Cu at (231.8, 247.5)
- added C2: 100nF, Capacitor_SMD:C_0603_1608Metric, B.Cu at (242.8, 247.5)
- added C3: 100nF, Capacitor_SMD:C_0603_1608Metric, B.Cu at (253.8, 247.5)
- added C4: 100nF, Capacitor_SMD:C_0603_1608Metric, B.Cu at (264.8, 247.5)
- added C5: 100nF, Capacitor_SMD:C_0603_1608Metric, B.Cu at (237.0, 176.5)
- added H1: M3, MountingHole:MountingHole_3.2mm_M3, F.Cu at (240.0, 259.5)
- added H2: M3, MountingHole:MountingHole_3.2mm_M3, F.Cu at (262.0, 259.5)
- added H3: M3, MountingHole:MountingHole_3.2mm_M3, F.Cu at (240.0, 175.5)
- added H4: M3, MountingHole:MountingHole_3.2mm_M3, F.Cu at (262.0, 175.5)
- added J1: to PCB-A (JST-SH 6), Connector_JST:JST_SH_SM06B-SRSS-TB_1x06-1MP_P1.00mm_Horizontal, B.Cu at (231.5, 176.5)
- added RV1: RS6011 B50K, groovepush:ALPS_RS6011P_60mm, F.Cu at (234.5, 217.5)
- added RV2: RS6011 B50K, groovepush:ALPS_RS6011P_60mm, F.Cu at (245.5, 217.5)
- added RV3: RS6011 B50K, groovepush:ALPS_RS6011P_60mm, F.Cu at (256.5, 217.5)
- added RV4: RS6011 B50K, groovepush:ALPS_RS6011P_60mm, F.Cu at (267.5, 217.5)
Routing:
- net /FADER4: track 0.00 -> 102.3 mm, vias 0 -> 1
- net /FADER3: track 0.00 -> 90.7 mm, vias 0 -> 1
- net /FADER2: track 0.00 -> 83.9 mm, vias 0 -> 1
- net /FADER1: track 0.00 -> 81.6 mm, vias 0 -> 1
- net /+3V3: track 0.00 -> 41.5 mm
- net /GND: track 0.00 -> 5.85 mm, vias 0 -> 86
- added copper zone on B.Cu, net /GND
- added copper zone on F.Cu, net /GND
Other:
- board outline added: 46 x 92 mm
