File: hardware/boards/pcb-f/pcb-f.kicad_sch (KiCad schematic)
At the start: 14 parts, among them J1 to PCB-A (JST-SH 6)

Commit message: hw(boards): all panel boards routed to DRC 0/0/0, add PCB-S shield adapter, fab outputs
PCB-A, PCB-F, PCB-K1, PCB-K2 and the new PCB-S pass DRC with schematic parity and ERC.
Single-sided bottom assembly; PCB-S ships bare (hand-soldered).

- PCB-A: MCP23017 0x20 moved to SSOP-28 in the front band between E4 and E5; J4 (to PCB-K1)
  moved to the tab next to J1 (cable ~20-25 cm) so the bus stays off the encoder strip;
  strip front edge 99 -> 97.5; H4 onto the tab.
- PCB-K1: MCP 0x21 pins reordered for a planar fan-out; U1 is SSOP-28; J2 over U2.
- PCB-S: shield adapter for the carrier's J15/J16 (I2C -> JST-SH 4, Serial5 -> JST-PH 4 to the M4).
- tools: grid router now sees footprint Edge.Cuts windows and exact pad keep-outs; finish_routing
  routes shortest-first, joins split nets and rips up endpoint blockers; new repair_routes.py and
  tie_loose_gnd.py; GND escapes respect the real outline; sync_from_netlist re-assigns pad nets;
  export_fab groups BOM lines per part and covers PCB-S.
- fab/: Gerbers, BOM and CPL per board for JLCPCB.

Co-Authored-By: Claude Sonnet 5.5 <noreply@anthropic.com>
Parts:
- C1, C2, C3, C4, C5: LCSC (none) -> C14663
- J1: LCSC (none) -> C160405
Changed lines of the file:
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@@
+			)
+		)
+		(property "LCSC" "C14663"
+			(at 49.53 90.17 0)
+			(hide yes)
+			(show_name no)
+			(do_not_autoplace no)
+			(effects
+				(font
+					(size 1.27 1.27)
+				)
 			)
 		)
@@
 			)
 		)
+		(property "LCSC" "C14663"
+			(at 80.01 90.17 0)
+			(hide yes)
+			(show_name no)
+			(do_not_autoplace no)
+			(effects
+				(font
+					(size 1.27 1.27)
+				)
+			)
+		)
 		(property "Description" "Unpolarized capacitor"
 			(at 80.01 90.17 0)
@@
 			)
 		)
+		(property "LCSC" "C14663"
+			(at 110.49 90.17 0)
+			(hide yes)
+			(show_name no)
+			(do_not_autoplace no)
+			(effects
+				(font
+					(size 1.27 1.27)
+				)
+			)
+		)
 		(property "Description" "Unpolarized capacitor"
 			(at 110.49 90.17 0)
@@
 			)
 		)
+		(property "LCSC" "C14663"
+			(at 139.7 90.17 0)
+			(hide yes)
+			(show_name no)
+			(do_not_autoplace no)
+			(effects
+				(font
+					(size 1.27 1.27)
+				)
+			)
+		)
 		(property "Description" "Unpolarized capacitor"
 			(at 139.7 90.17 0)
@@
 			)
 		)
+		(property "LCSC" "C14663"
+			(at 170.18 90.17 0)
+			(hide yes)
+			(show_name no)
+			(do_not_autoplace no)
+			(effects
+				(font
+					(size 1.27 1.27)
+				)
+			)
+		)
 		(property "Description" "Unpolarized capacitor"
 			(at 170.18 90.17 0)
@@
 			(at 199.39 59.69 0)
 			(hide yes)
+			(show_name no)
+			(do_not_autoplace no)
+			(effects
+				(font
+					(size 1.27 1.27)
+				)
+			)
+		)
+		(property "LCSC" "C160405"
+			(at 199.39 59.69 0)
+			(hide yes)
