File: hardware/boards/pcb-k1/pcb-k1.kicad_pcb (KiCad board)
At the start: 2 copper layers, 0 parts

Commit message: hw(boards): PCB-F and PCB-K2 placed and routed, DRC 0/0/0 with schematic parity
Placement from panel-coordinates.csv (shared frame for all boards), Brain
board tools reused (route_board/finish_routing/add_gnd_escapes/pours/fields),
plus sync_from_netlist.py (MCP sync drops the '/' net prefix and BOM attrs)
and build.sh to rebuild a board end to end. LED-window DRC rule copied
from the Brain's PCB-K.

Co-Authored-By: Claude Opus 5.5 <noreply@anthropic.com>
Parts:
- added C1, C10, C11, C12, C13, C14, C15, C16, C17, C18, C19, C2, C20, C21, C22, C23, C24: 100nF, Capacitor_SMD:C_0603_1608Metric, F.Cu at (0.00, 0.00)
- added C3: 47uF, Capacitor_SMD:C_1206_3216Metric, F.Cu at (0.00, 0.00)
- added D1: SK6812MINI-EA (QUANTIZE, idx 5), LED_SMD:LED_SK6812MINI-E_3.2x2.8mm_P1.5mm_ReverseMount, F.Cu at (0.00, 0.00)
- added D10: SK6812MINI-EA (LOOP, idx 14), LED_SMD:LED_SK6812MINI-E_3.2x2.8mm_P1.5mm_ReverseMount, F.Cu at (0.00, 0.00)
- added D11: SK6812MINI-EA (METRO, idx 15), LED_SMD:LED_SK6812MINI-E_3.2x2.8mm_P1.5mm_ReverseMount, F.Cu at (0.00, 0.00)
- added D12: SK6812MINI-EA (BANK_L, idx 16), LED_SMD:LED_SK6812MINI-E_3.2x2.8mm_P1.5mm_ReverseMount, F.Cu at (0.00, 0.00)
- added D13: SK6812MINI-EA (BANK_R, idx 17), LED_SMD:LED_SK6812MINI-E_3.2x2.8mm_P1.5mm_ReverseMount, F.Cu at (0.00, 0.00)
- added D14: SK6812MINI-EA (OCT_DN, idx 18), LED_SMD:LED_SK6812MINI-E_3.2x2.8mm_P1.5mm_ReverseMount, F.Cu at (0.00, 0.00)
- added D15: SK6812MINI-EA (OCT_UP, idx 19), LED_SMD:LED_SK6812MINI-E_3.2x2.8mm_P1.5mm_ReverseMount, F.Cu at (0.00, 0.00)
- added D2: SK6812MINI-EA (DUPLICATE, idx 6), LED_SMD:LED_SK6812MINI-E_3.2x2.8mm_P1.5mm_ReverseMount, F.Cu at (0.00, 0.00)
- added D3: SK6812MINI-EA (DELETE, idx 7), LED_SMD:LED_SK6812MINI-E_3.2x2.8mm_P1.5mm_ReverseMount, F.Cu at (0.00, 0.00)
- added D4: SK6812MINI-EA (UNDO, idx 8), LED_SMD:LED_SK6812MINI-E_3.2x2.8mm_P1.5mm_ReverseMount, F.Cu at (0.00, 0.00)
- added D5: SK6812MINI-EA (NEW, idx 9), LED_SMD:LED_SK6812MINI-E_3.2x2.8mm_P1.5mm_ReverseMount, F.Cu at (0.00, 0.00)
- added D6: SK6812MINI-EA (SHIFT, idx 10), LED_SMD:LED_SK6812MINI-E_3.2x2.8mm_P1.5mm_ReverseMount, F.Cu at (0.00, 0.00)
- added D7: SK6812MINI-EA (PLAY, idx 11), LED_SMD:LED_SK6812MINI-E_3.2x2.8mm_P1.5mm_ReverseMount, F.Cu at (0.00, 0.00)
- added D8: SK6812MINI-EA (STOP, idx 12), LED_SMD:LED_SK6812MINI-E_3.2x2.8mm_P1.5mm_ReverseMount, F.Cu at (0.00, 0.00)
- added D9: SK6812MINI-EA (RECORD, idx 13), LED_SMD:LED_SK6812MINI-E_3.2x2.8mm_P1.5mm_ReverseMount, F.Cu at (0.00, 0.00)
- added H1, H2, H3, H4: M3, MountingHole:MountingHole_3.2mm_M3, F.Cu at (0.00, 0.00)
- added J1: from PCB-A J4 (JST-SH 10), Connector_JST:JST_SH_SM10B-SRSS-TB_1x10-1MP_P1.00mm_Horizontal, F.Cu at (0.00, 0.00)
- added J2: to PCB-K2 J1 (JST-SH 10), Connector_JST:JST_SH_SM10B-SRSS-TB_1x10-1MP_P1.00mm_Horizontal, F.Cu at (0.00, 0.00)
- added R1: 10k, Resistor_SMD:R_0603_1608Metric, F.Cu at (0.00, 0.00)
- added SW1: QUANTIZE, groovepush:SW_Kailh_Choc_V2_1u, F.Cu at (0.00, 0.00)
- added SW10: LOOP, groovepush:SW_Kailh_Choc_V2_1u, F.Cu at (0.00, 0.00)
- added SW11: METRO, groovepush:SW_Kailh_Choc_V2_1u, F.Cu at (0.00, 0.00)
- added SW12: BANK_L, groovepush:SW_Kailh_Choc_V2_1u, F.Cu at (0.00, 0.00)
- added SW13: BANK_R, groovepush:SW_Kailh_Choc_V2_1u, F.Cu at (0.00, 0.00)
- added SW14: OCT_DN, groovepush:SW_Kailh_Choc_V2_1u, F.Cu at (0.00, 0.00)
- added SW15: OCT_UP, groovepush:SW_Kailh_Choc_V2_1u, F.Cu at (0.00, 0.00)
- added SW2: DUPLICATE, groovepush:SW_Kailh_Choc_V2_1u, F.Cu at (0.00, 0.00)
- added SW3: DELETE, groovepush:SW_Kailh_Choc_V2_1u, F.Cu at (0.00, 0.00)
- added SW4: UNDO, groovepush:SW_Kailh_Choc_V2_1u, F.Cu at (0.00, 0.00)
- added SW5: NEW, groovepush:SW_Kailh_Choc_V2_1u, F.Cu at (0.00, 0.00)
- added SW6: SHIFT, groovepush:SW_Kailh_Choc_V2_1u, F.Cu at (0.00, 0.00)
- added SW7: PLAY, groovepush:SW_Kailh_Choc_V2_1u, F.Cu at (0.00, 0.00)
- added SW8: STOP, groovepush:SW_Kailh_Choc_V2_1u, F.Cu at (0.00, 0.00)
- added SW9: RECORD, groovepush:SW_Kailh_Choc_V2_1u, F.Cu at (0.00, 0.00)
- added U1: MCP23017-E/SO @0x21, Package_SO:SOIC-28W_7.5x17.9mm_P1.27mm, F.Cu at (0.00, 0.00)
- added U2: MCP23017-E/SO @0x22, Package_SO:SOIC-28W_7.5x17.9mm_P1.27mm, F.Cu at (0.00, 0.00)
Other:
- board outline added: 3.6 x 3.2 mm

Commit message: hw(boards): all panel boards routed to DRC 0/0/0, add PCB-S shield adapter, fab outputs
PCB-A, PCB-F, PCB-K1, PCB-K2 and the new PCB-S pass DRC with schematic parity and ERC.
Single-sided bottom assembly; PCB-S ships bare (hand-soldered).

- PCB-A: MCP23017 0x20 moved to SSOP-28 in the front band between E4 and E5; J4 (to PCB-K1)
  moved to the tab next to J1 (cable ~20-25 cm) so the bus stays off the encoder strip;
  strip front edge 99 -> 97.5; H4 onto the tab.
- PCB-K1: MCP 0x21 pins reordered for a planar fan-out; U1 is SSOP-28; J2 over U2.
- PCB-S: shield adapter for the carrier's J15/J16 (I2C -> JST-SH 4, Serial5 -> JST-PH 4 to the M4).
- tools: grid router now sees footprint Edge.Cuts windows and exact pad keep-outs; finish_routing
  routes shortest-first, joins split nets and rips up endpoint blockers; new repair_routes.py and
  tie_loose_gnd.py; GND escapes respect the real outline; sync_from_netlist re-assigns pad nets;
  export_fab groups BOM lines per part and covers PCB-S.
- fab/: Gerbers, BOM and CPL per board for JLCPCB.

Co-Authored-By: Claude Sonnet 5.5 <noreply@anthropic.com>
Parts:
- removed H3, H4: M3, MountingHole:MountingHole_3.2mm_M3
- C1, C10, C11, C12, C13, C14, C15, C16, C17, C18, C19, C2, C20, C21, C22, C23, C24, C3, D1, D10, D11, D12, D13, D14, D15, D2, D3, D4, D5, D6, D7, D8, D9, J1, J2, R1, U2: moved to B.Cu
- U1: value MCP23017-E/SO @0x21 -> MCP23017T-E/SS @0x21; footprint Package_SO:SOIC-28W_7.5x17.9mm_P1.27mm -> Package_SO:SSOP-28_5.3x10.2mm_P0.65mm; moved to B.Cu
- moved C24 346.6 mm to (228.0, 261.1), turned to 90 degrees
- moved SW15 345.5 mm to (220.5, 266.0)
- moved D15 341.7 mm to (220.5, 261.1)
- moved C23 334.1 mm to (208.5, 261.1), turned to 90 degrees
- moved SW14 333.4 mm to (201.0, 266.0)
- moved D14 329.5 mm to (201.0, 261.1)
- moved C22 322.3 mm to (189.0, 261.1), turned to 90 degrees
- moved SW13 322.0 mm to (181.5, 266.0)
- moved D13 318.0 mm to (181.5, 261.1)
- moved SW12 311.4 mm to (162.0, 266.0)
- moved C21 311.3 mm to (169.5, 261.1), turned to 90 degrees
- moved D12 307.2 mm to (162.0, 261.1)
- moved U1 305.0 mm to (149.2, 266.0)
- moved SW11 299.0 mm to (136.5, 266.0)
- moved C1 298.9 mm to (149.2, 259.0)
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Connections:
- net +3V3 renamed /+3V3
- net +5V renamed /+5V
- net GND renamed /GND
- net INT_K renamed /INT_K
- net KEY_BROWSE renamed /KEY_BROWSE
- net KEY_DEVICE renamed /KEY_DEVICE
- net KEY_MIX renamed /KEY_MIX
- net KEY_NOTE renamed /KEY_NOTE
- net KEY_SESSION renamed /KEY_SESSION
- net KEY_UNDO renamed /KEY_UNDO
- net LED_1 renamed /LED_1
- net LED_10 renamed /LED_10
- net LED_11 renamed /LED_11
- net LED_12 renamed /LED_12
- net LED_13 renamed /LED_13
- net LED_14 renamed /LED_14
- net LED_2 renamed /LED_2
- net LED_3 renamed /LED_3
- net LED_4 renamed /LED_4
- net LED_5 renamed /LED_5
- net LED_6 renamed /LED_6
- net LED_7 renamed /LED_7
- net LED_8 renamed /LED_8
- net LED_9 renamed /LED_9
- net LED_DIN renamed /LED_DIN
- net LED_END renamed /LED_END
- net LED_K2_RET renamed /LED_K2_RET
- net SCL renamed /SCL
- net SDA renamed /SDA
- SW1 pad 1: KEY_QUANTIZE -> /KEY_QUANTIZE
- SW10 pad 1: KEY_LOOP -> /KEY_LOOP
- SW11 pad 1: KEY_METRO -> /KEY_METRO
- SW12 pad 1: KEY_BANK_L -> /KEY_BANK_L
- SW13 pad 1: KEY_BANK_R -> /KEY_BANK_R
- SW14 pad 1: KEY_OCT_DN -> /KEY_OCT_DN
- SW15 pad 1: KEY_OCT_UP -> /KEY_OCT_UP
- SW2 pad 1: KEY_DUPLICATE -> /KEY_DUPLICATE
- SW3 pad 1: KEY_DELETE -> /KEY_DELETE
- SW5 pad 1: KEY_NEW -> /KEY_NEW
- SW6 pad 1: KEY_SHIFT -> /KEY_SHIFT
- SW7 pad 1: KEY_PLAY -> /KEY_PLAY
- SW8 pad 1: KEY_STOP -> /KEY_STOP
- SW9 pad 1: KEY_RECORD -> /KEY_RECORD
- U1 pad 1: KEY_BANK_R -> /KEY_METRO
- U1 pad 11: (no net) -> unconnected-(U1-NC-Pad11)
- U1 pad 14: (no net) -> unconnected-(U1-NC-Pad14)
- U1 pad 19: (no net) -> unconnected-(U1-INTB-Pad19)
- U1 pad 2: KEY_OCT_DN -> /KEY_LOOP
- U1 pad 21: KEY_PLAY -> /KEY_OCT_UP
- U1 pad 22: KEY_STOP -> /KEY_OCT_DN
- U1 pad 23: KEY_RECORD -> /KEY_BANK_R
- U1 pad 24: KEY_LOOP -> /KEY_BANK_L
- U1 pad 25: KEY_METRO -> unconnected-(U1-GPA4-Pad25)
- U1 pad 26: KEY_SHIFT -> unconnected-(U1-GPA5-Pad26)
- U1 pad 27: KEY_BANK_L -> unconnected-(U1-GPA6-Pad27)
- U1 pad 28: (no net) -> unconnected-(U1-GPA7-Pad28)
- U1 pad 3: KEY_OCT_UP -> /KEY_RECORD
- U1 pad 4: KEY_DELETE -> /KEY_STOP
- U1 pad 5: KEY_DUPLICATE -> /KEY_PLAY
- U1 pad 6: KEY_QUANTIZE -> unconnected-(U1-GPB5-Pad6)
- U1 pad 7: KEY_NEW -> unconnected-(U1-GPB6-Pad7)
- U1 pad 8: (no net) -> unconnected-(U1-GPB7-Pad8)
- U2 pad 1: (no net) -> /KEY_DELETE
- U2 pad 11: (no net) -> unconnected-(U2-NC-Pad11)
- U2 pad 14: (no net) -> unconnected-(U2-NC-Pad14)
- U2 pad 19: (no net) -> unconnected-(U2-INTB-Pad19)
- U2 pad 2: (no net) -> /KEY_DUPLICATE
- U2 pad 27: (no net) -> /KEY_SHIFT
- U2 pad 28: (no net) -> unconnected-(U2-GPA7-Pad28)
- U2 pad 3: (no net) -> /KEY_QUANTIZE
- U2 pad 4: (no net) -> /KEY_NEW
- U2 pad 5: (no net) -> unconnected-(U2-GPB4-Pad5)
- U2 pad 6: (no net) -> unconnected-(U2-GPB5-Pad6)
- U2 pad 7: (no net) -> unconnected-(U2-GPB6-Pad7)
- U2 pad 8: (no net) -> unconnected-(U2-GPB7-Pad8)
Routing:
- net /+5V: track 0.00 -> 471.4 mm, vias 0 -> 10
- net /+3V3: track 0.00 -> 238.8 mm, vias 0 -> 4
- net /SCL: track 0.00 -> 202.8 mm
- net /INT_K: track 0.00 -> 197.4 mm, vias 0 -> 8
- net /SDA: track 0.00 -> 191.8 mm, vias 0 -> 6
- net /KEY_PLAY: track 0.00 -> 94.8 mm
- net /KEY_SHIFT: track 0.00 -> 82.8 mm, vias 0 -> 1
- net /KEY_OCT_UP: track 0.00 -> 73.8 mm, vias 0 -> 1
- net /KEY_STOP: track 0.00 -> 70.2 mm, vias 0 -> 1
- net /KEY_OCT_DN: track 0.00 -> 57.0 mm
- net /GND: track 0.00 -> 51.4 mm, vias 0 -> 152
- net /KEY_RECORD: track 0.00 -> 49.9 mm
- net /KEY_DELETE: track 0.00 -> 49.8 mm, vias 0 -> 1
- net /LED_5: track 0.00 -> 46.4 mm
- net /LED_3: track 0.00 -> 40.9 mm, vias 0 -> 2
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- added copper zone on B.Cu, net /GND
- added copper zone on F.Cu, net /GND
Other:
- board size 3.6 x 3.2 mm -> 207.5 x 91 mm
