File: hardware/boards/pcb-k1/pcb-k1.kicad_sch (KiCad schematic)
At the start: 57 parts, among them J1 from PCB-A J4 (JST-SH 10), J2 to PCB-K2 J1 (JST-SH 10), SW1 QUANTIZE, SW10 LOOP, SW11 METRO, SW12 BANK_L, SW13 BANK_R, SW14 OCT_DN, SW15 OCT_UP, SW2 DUPLICATE, SW3 DELETE, SW4 UNDO, SW5 NEW, SW6 SHIFT, SW7 PLAY, SW8 STOP, SW9 RECORD, U1 MCP23017-E/SO @0x21, U2 MCP23017-E/SO @0x22

Commit message: hw(boards): all panel boards routed to DRC 0/0/0, add PCB-S shield adapter, fab outputs
PCB-A, PCB-F, PCB-K1, PCB-K2 and the new PCB-S pass DRC with schematic parity and ERC.
Single-sided bottom assembly; PCB-S ships bare (hand-soldered).

- PCB-A: MCP23017 0x20 moved to SSOP-28 in the front band between E4 and E5; J4 (to PCB-K1)
  moved to the tab next to J1 (cable ~20-25 cm) so the bus stays off the encoder strip;
  strip front edge 99 -> 97.5; H4 onto the tab.
- PCB-K1: MCP 0x21 pins reordered for a planar fan-out; U1 is SSOP-28; J2 over U2.
- PCB-S: shield adapter for the carrier's J15/J16 (I2C -> JST-SH 4, Serial5 -> JST-PH 4 to the M4).
- tools: grid router now sees footprint Edge.Cuts windows and exact pad keep-outs; finish_routing
  routes shortest-first, joins split nets and rips up endpoint blockers; new repair_routes.py and
  tie_loose_gnd.py; GND escapes respect the real outline; sync_from_netlist re-assigns pad nets;
  export_fab groups BOM lines per part and covers PCB-S.
- fab/: Gerbers, BOM and CPL per board for JLCPCB.

Co-Authored-By: Claude Sonnet 5.5 <noreply@anthropic.com>
Parts:
- removed H3, H4: M3, MountingHole:MountingHole_3.2mm_M3, symbol Mechanical:MountingHole
- removed U1: MCP23017-E/SO @0x21, Package_SO:SOIC-28W_7.5x17.9mm_P1.27mm, symbol Interface_Expansion:MCP23017x-x-SO
- added U1: MCP23017T-E/SS @0x21, Package_SO:SSOP-28_5.3x10.2mm_P0.65mm, symbol Interface_Expansion:MCP23017x-x-SS
- C1, C10, C11, C12, C13, C14, C15, C16, C17, C18, C19, C2, C20, C21, C22, C23, C24: LCSC (none) -> C14663
- C3: LCSC (none) -> C96123
- D1, D10, D11, D12, D13, D14, D15, D2, D3, D4, D5, D6, D7, D8, D9: LCSC (none) -> C5378731
- J1, J2: LCSC (none) -> C160409
- R1: LCSC (none) -> C25804
- U2: LCSC (none) -> C47023
Connections:
- net +3V3: now also U1.15 (A0), U1.18 (~{RESET}), U1.9 (V_{DD})
- net GND: now also U1.10 (V_{SS}), U1.16 (A1), U1.17 (A2)
- net INT_K: now also U1.20 (INTA)
- net KEY_BANK_L: now also U1.24 (GPA3)
- net KEY_BANK_R: now also U1.23 (GPA2)
- net KEY_DELETE: now also U2.1 (GPB0)
- net KEY_DUPLICATE: now also U2.2 (GPB1)
- net KEY_LOOP: now also U1.2 (GPB1)
- net KEY_METRO: now also U1.1 (GPB0)
- net KEY_NEW: now also U2.4 (GPB3)
- net KEY_OCT_DN: now also U1.22 (GPA1)
- net KEY_OCT_UP: now also U1.21 (GPA0)
- net KEY_PLAY: now also U1.5 (GPB4)
- net KEY_QUANTIZE: now also U2.3 (GPB2)
- net KEY_RECORD: now also U1.3 (GPB2)
- net KEY_SHIFT: now also U2.27 (GPA6)
- net KEY_STOP: now also U1.4 (GPB3)
- net SCL: now also U1.12 (SCK)
- net SDA: now also U1.13 (SDA)
