File: hardware/boards/pcb-k2/pcb-k2.kicad_pcb (KiCad board)
At the start: 2 copper layers, 0 parts

Commit message: hw(boards): PCB-F and PCB-K2 placed and routed, DRC 0/0/0 with schematic parity
Placement from panel-coordinates.csv (shared frame for all boards), Brain
board tools reused (route_board/finish_routing/add_gnd_escapes/pours/fields),
plus sync_from_netlist.py (MCP sync drops the '/' net prefix and BOM attrs)
and build.sh to rebuild a board end to end. LED-window DRC rule copied
from the Brain's PCB-K.

Co-Authored-By: Claude Opus 5.5 <noreply@anthropic.com>
Parts:
- added C1: 47uF, Capacitor_SMD:C_1206_3216Metric, B.Cu at (26.5, 160.5)
- added C10: 100nF, Capacitor_SMD:C_0603_1608Metric, B.Cu at (13.5, 150.1)
- added C11: 100nF, Capacitor_SMD:C_0603_1608Metric, B.Cu at (13.5, 131.6)
- added C12: 100nF, Capacitor_SMD:C_0603_1608Metric, B.Cu at (13.5, 113.1)
- added C13: 100nF, Capacitor_SMD:C_0603_1608Metric, B.Cu at (13.5, 94.6)
- added C14: 100nF, Capacitor_SMD:C_0603_1608Metric, B.Cu at (13.5, 76.1)
- added D1: SK6812MINI-EA (BROWSE, idx 0), LED_SMD:LED_SK6812MINI-E_3.2x2.8mm_P1.5mm_ReverseMount, B.Cu at (21.0, 150.1)
- added D2: SK6812MINI-EA (MIX, idx 1), LED_SMD:LED_SK6812MINI-E_3.2x2.8mm_P1.5mm_ReverseMount, B.Cu at (21.0, 131.6)
- added D3: SK6812MINI-EA (DEVICE, idx 2), LED_SMD:LED_SK6812MINI-E_3.2x2.8mm_P1.5mm_ReverseMount, B.Cu at (21.0, 113.1)
- added D4: SK6812MINI-EA (NOTE, idx 3), LED_SMD:LED_SK6812MINI-E_3.2x2.8mm_P1.5mm_ReverseMount, B.Cu at (21.0, 94.6)
- added D5: SK6812MINI-EA (SESSION, idx 4), LED_SMD:LED_SK6812MINI-E_3.2x2.8mm_P1.5mm_ReverseMount, B.Cu at (21.0, 76.1)
- added H1: M2.5, MountingHole:MountingHole_2.7mm_M2.5, F.Cu at (15.5, 69.5)
- added H2: M2.5, MountingHole:MountingHole_2.7mm_M2.5, F.Cu at (26.0, 69.5)
- added J1: from PCB-K1 J2 (JST-SH 10), Connector_JST:JST_SH_SM10B-SRSS-TB_1x10-1MP_P1.00mm_Horizontal, B.Cu at (21.0, 166.2)
- added SW1: BROWSE, groovepush:SW_Kailh_Choc_V2_1u, F.Cu at (21.0, 155.0)
- added SW2: MIX, groovepush:SW_Kailh_Choc_V2_1u, F.Cu at (21.0, 136.5)
- added SW3: DEVICE, groovepush:SW_Kailh_Choc_V2_1u, F.Cu at (21.0, 118.0)
- added SW4: NOTE, groovepush:SW_Kailh_Choc_V2_1u, F.Cu at (21.0, 99.5)
- added SW5: SESSION, groovepush:SW_Kailh_Choc_V2_1u, F.Cu at (21.0, 81.0)
Routing:
- net /+5V: track 0.00 -> 195.5 mm, vias 0 -> 3
- net /LED_K2_RET: track 0.00 -> 100.5 mm, vias 0 -> 2
- net /KEY_SESSION: track 0.00 -> 82.9 mm, vias 0 -> 1
- net /KEY_NOTE: track 0.00 -> 67.4 mm, vias 0 -> 1
- net /KEY_DEVICE: track 0.00 -> 45.3 mm, vias 0 -> 1
- net /LED_4: track 0.00 -> 37.8 mm
- net /KEY_MIX: track 0.00 -> 24.3 mm, vias 0 -> 1
- net /LED_2: track 0.00 -> 19.7 mm
- net /LED_1: track 0.00 -> 19.7 mm
- net /LED_3: track 0.00 -> 19.6 mm
- net /LED_DIN: track 0.00 -> 17.3 mm
- net /GND: track 0.00 -> 14.4 mm, vias 0 -> 26
- net /KEY_BROWSE: track 0.00 -> 3.51 mm
- added copper zone on B.Cu, net /GND
- added copper zone on F.Cu, net /GND
Other:
- board outline added: 18.5 x 103.5 mm
