File: hardware/boards/pcb-k2/pcb-k2.kicad_sch (KiCad schematic)
At the start: 19 parts, among them J1 from PCB-K1 J2 (JST-SH 10), SW1 BROWSE, SW2 MIX, SW3 DEVICE, SW4 NOTE, SW5 SESSION

Commit message: hw(boards): all panel boards routed to DRC 0/0/0, add PCB-S shield adapter, fab outputs
PCB-A, PCB-F, PCB-K1, PCB-K2 and the new PCB-S pass DRC with schematic parity and ERC.
Single-sided bottom assembly; PCB-S ships bare (hand-soldered).

- PCB-A: MCP23017 0x20 moved to SSOP-28 in the front band between E4 and E5; J4 (to PCB-K1)
  moved to the tab next to J1 (cable ~20-25 cm) so the bus stays off the encoder strip;
  strip front edge 99 -> 97.5; H4 onto the tab.
- PCB-K1: MCP 0x21 pins reordered for a planar fan-out; U1 is SSOP-28; J2 over U2.
- PCB-S: shield adapter for the carrier's J15/J16 (I2C -> JST-SH 4, Serial5 -> JST-PH 4 to the M4).
- tools: grid router now sees footprint Edge.Cuts windows and exact pad keep-outs; finish_routing
  routes shortest-first, joins split nets and rips up endpoint blockers; new repair_routes.py and
  tie_loose_gnd.py; GND escapes respect the real outline; sync_from_netlist re-assigns pad nets;
  export_fab groups BOM lines per part and covers PCB-S.
- fab/: Gerbers, BOM and CPL per board for JLCPCB.

Co-Authored-By: Claude Sonnet 5.5 <noreply@anthropic.com>
Parts:
- C1: LCSC (none) -> C96123
- C10, C11, C12, C13, C14: LCSC (none) -> C14663
- D1, D2, D3, D4, D5: LCSC (none) -> C5378731
- J1: LCSC (none) -> C160409
Changed lines of the file:
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@@
+			)
+		)
+		(property "LCSC" "C160409"
+			(at 30.48 59.69 0)
+			(hide yes)
+			(show_name no)
+			(do_not_autoplace no)
+			(effects
+				(font
+					(size 1.27 1.27)
+				)
 			)
 		)
@@
 			)
 		)
+		(property "LCSC" "C96123"
+			(at 59.69 39.37 0)
+			(hide yes)
+			(show_name no)
+			(do_not_autoplace no)
+			(effects
+				(font
+					(size 1.27 1.27)
+				)
+			)
+		)
 		(property "Description" "Unpolarized capacitor"
 			(at 59.69 39.37 0)
@@
 			)
 		)
+		(property "LCSC" "C5378731"
+			(at 100.33 64.77 0)
+			(hide yes)
+			(show_name no)
+			(do_not_autoplace no)
+			(effects
+				(font
+					(size 1.27 1.27)
+				)
+			)
+		)
 		(property "Description" "RGB LED with integrated controller"
 			(at 100.33 64.77 0)
@@
 			)
 		)
+		(property "LCSC" "C14663"
+			(at 115.57 64.77 0)
+			(hide yes)
+			(show_name no)
+			(do_not_autoplace no)
+			(effects
+				(font
+					(size 1.27 1.27)
+				)
+			)
+		)
 		(property "Description" "Unpolarized capacitor"
 			(at 115.57 64.77 0)
@@
 			)
 		)
+		(property "LCSC" "C5378731"
+			(at 139.7 64.77 0)
+			(hide yes)
+			(show_name no)
+			(do_not_autoplace no)
+			(effects
+				(font
+					(size 1.27 1.27)
+				)
+			)
+		)
 		(property "Description" "RGB LED with integrated controller"
 			(at 139.7 64.77 0)
@@
 			)
 		)
+		(property "LCSC" "C14663"
+			(at 154.94 64.77 0)
+			(hide yes)
+			(show_name no)
+			(do_not_autoplace no)
+			(effects
+				(font
+					(size 1.27 1.27)
+				)
+			)
+		)
 		(property "Description" "Unpolarized capacitor"
 			(at 154.94 64.77 0)
@@
 			)
 		)
+		(property "LCSC" "C5378731"
+			(at 180.34 64.77 0)
+			(hide yes)
+			(show_name no)
+			(do_not_autoplace no)
+			(effects
+				(font
+					(size 1.27 1.27)
+				)
+			)
+		)
 		(property "Description" "RGB LED with integrated controller"
 			(at 180.34 64.77 0)
@@
 			)
 		)
+		(property "LCSC" "C14663"
+			(at 195.58 64.77 0)
+			(hide yes)
+			(show_name no)
+			(do_not_autoplace no)
+			(effects
+				(font
+					(size 1.27 1.27)
+				)
+			)
+		)
 		(property "Description" "Unpolarized capacitor"
 			(at 195.58 64.77 0)
@@
 			)
 		)
+		(property "LCSC" "C5378731"
+			(at 219.71 64.77 0)
+			(hide yes)
+			(show_name no)
+			(do_not_autoplace no)
+			(effects
+				(font
+					(size 1.27 1.27)
+				)
+			)
+		)
 		(property "Description" "RGB LED with integrated controller"
 			(at 219.71 64.77 0)
@@
 			)
 		)
+		(property "LCSC" "C14663"
+			(at 234.95 64.77 0)
+			(hide yes)
+			(show_name no)
+			(do_not_autoplace no)
+			(effects
+				(font
+					(size 1.27 1.27)
+				)
+			)
+		)
 		(property "Description" "Unpolarized capacitor"
 			(at 234.95 64.77 0)
@@
 			)
 		)
+		(property "LCSC" "C5378731"
+			(at 260.35 64.77 0)
+			(hide yes)
+			(show_name no)
+			(do_not_autoplace no)
+			(effects
+				(font
+					(size 1.27 1.27)
+				)
+			)
+		)
 		(property "Description" "RGB LED with integrated controller"
 			(at 260.35 64.77 0)
@@
 			(at 275.59 64.77 0)
 			(hide yes)
+			(show_name no)
+			(do_not_autoplace no)
+			(effects
+				(font
+					(size 1.27 1.27)
+				)
+			)
+		)
+		(property "LCSC" "C14663"
+			(at 275.59 64.77 0)
+			(hide yes)
